Commit message: renamed base_link_ground to base_link to simplify TF tree

File: coco_one.urdf (robot description, URDF)
Before this commit: robot coco_one, 1 links, 0 joints
Links:
- removed link base_link_ground
- added link base_link; visual mesh filename=https://raw.githubusercontent.com/cocorobotics/coco_model/m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 scale=0.001 0.001 0.001

Commit message: update link name

File: coco_one.urdf (robot description, URDF)
Before this commit: robot coco_one, 1 links, 0 joints
Links:
- removed link base_link
- added link base_link_ground; visual mesh filename=https://raw.githubusercontent.com/cocorobotics/coco_model/m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 scale=0.001 0.001 0.001
